Commit message: update README.md

File: urdf/cam.SLDASM.urdf (robot description, URDF)
Before this commit: robot hit_mechanism2, 4 links, 3 joints
Links:
- removed link link1
- added link link3, mass 0.0149225651045515; collision mesh filename=package://cam.SLDASM/meshes/link3.STL; visual mesh filename=package://cam.SLDASM/meshes/link3.STL
- added link link4, mass 0.00468304605147202; collision mesh filename=package://cam.SLDASM/meshes/link4.STL; visual mesh filename=package://cam.SLDASM/meshes/link4.STL
- link base_link: geometry collision mesh filename=package://cam.SLDASM/meshes/base_link.STL; visual mesh filename=package://cam.SLDASM/meshes/base_link.STL
- link cam_link: mass 0.123418384619757 -> 0.0932420859273589; geometry collision mesh filename=package://cam.SLDASM/meshes/cam_link.STL; visual mesh filename=package://cam.SLDASM/meshes/cam_link.STL
- link link2: mass 0.00285884931476671 -> 0.0157169361063451; geometry collision mesh filename=package://cam.SLDASM/meshes/link2.STL; visual mesh filename=package://cam.SLDASM/meshes/link2.STL
Joints:
- added joint joint4: type fixed, parent base_link, child link4, origin xyz=-0.0098346 0.0020564 0.00068033 rpy=1.5708 0 0, axis 0 0 0
- joint joint1: origin xyz=0 0 0 rpy=1.5708 0 0 -> xyz=0.0051654 -0.0081691 -0.1477 rpy=1.5708 0.0054199 0
- joint joint2: child link1 -> link2; limit lower=25 upper=55 effort=0 velocity=0 -> lower=0 upper=0 effort=0 velocity=0; origin xyz=-0.0130168913709829 0.00999999999999955 0.0350812000102613 rpy=1.5707963267949 0 0 -> xyz=-0.0078263 0.0018309 0.049232 rpy=1.5708 0 0
- joint joint3: child link2 -> link3; origin xyz=0.00299163531431282 0.00299170343325255 0.01 rpy=0 0 0 -> xyz=0.0029916 -0.15408 0.01 rpy=0 0 -0.12045; parent link1 -> link2
